Commit message: Zipper scaled and working

File: larc_robot_description/urdf/larc_robot_description.urdf (robot description, URDF)
Before this commit: robot larc_robot_description, 11 links, 10 joints
Joints:
- joint elbow: axis 1 0 0 -> -1 0 0

Commit message: Dynamixel library fixed

File: larc_robot_description/urdf/larc_robot_description.urdf (robot description, URDF)
Before this commit: robot larc_robot_description, 11 links, 10 joints
Joints:
- joint elbow: limit lower=-2.6 upper=2.6 effort=3.1 velocity=7 -> lower=-1.8 upper=1.7 effort=3.1 velocity=7
- joint shoulder: limit lower=-2.6 upper=2.6 effort=3.1 velocity=7 -> lower=-1.38 upper=1.1 effort=3.1 velocity=7

Commit message: Control funcionando una belleza

File: larc_robot_description/urdf/larc_robot_description.urdf (robot description, URDF)
Before this commit: robot larc_robot_description, 11 links, 10 joints
Joints:
- joint shoulder: limit lower=-1.38 upper=1.1 effort=3.1 velocity=7 -> lower=-1.9 upper=1.1 effort=3.1 velocity=7

Commit message: Backup 1

File: larc_robot_description/urdf/larc_robot_description.urdf (robot description, URDF)
Before this commit: robot larc_robot_description, 11 links, 10 joints
Joints:
- joint elbow: limit lower=-1.8 upper=1.7 effort=3.1 velocity=7 -> lower=-1.93 upper=1.93 effort=3.1 velocity=7

Commit message: Backup 2

File: larc_robot_description/urdf/larc_robot_description.urdf (robot description, URDF)
Before this commit: robot larc_robot_description, 11 links, 10 joints
Joints:
- joint zipper: limit lower=0.0 upper=0.16 effort=3.1 velocity=7 -> lower=0.0 upper=0.20 effort=3.1 velocity=7

Commit message: Backup 3

File: larc_robot_description/urdf/larc_robot_description.urdf (robot description, URDF)
Before this commit: robot larc_robot_description, 11 links, 10 joints
Joints:
- joint shoulder: limit lower=-1.9 upper=1.1 effort=3.1 velocity=7 -> lower=-1.9 upper=1.2 effort=3.1 velocity=7

Commit message: Final Version

File: larc_robot_description/urdf/larc_robot_description.urdf (robot description, URDF)
Before this commit: robot larc_robot_description, 11 links, 10 joints
Joints:
- joint zipper: limit lower=0.0 upper=0.20 effort=3.1 velocity=7 -> lower=0.0 upper=0.21 effort=3.1 velocity=3
